File: Antares-Transmitter.kicad_pcb (KiCad board)
At the start: 2 copper layers, 94 x 60.8 mm, 97 parts, among them J1001 Debugger Pin, J1101 Conn_01x02, J401 Conn_01x11, J501 Conn_01x03, J601 Conn_01x05, J602 Conn_01x06, J901 Conn_01x05, SW701 DOWN, SW702 UP, U201 STM32G070KBTx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

Commit message: :package: finished version 1.0.0, generated production files
Parts:
- added kibuzzard-66C9DF62: G***, kibuzzard-66C9DF62, F.Cu at (151.0, 108.0)
- added kibuzzard-66C9DFEC: G***, kibuzzard-66C9DFEC, B.Cu at (136.2, 132.6)
- added kibuzzard-66C9E01B: G***, kibuzzard-66C9E01B, B.Cu at (136.0, 107.6)
- added kibuzzard-66C9E05B: G***, kibuzzard-66C9E05B, B.Cu at (158.6, 126.0)
- added kibuzzard-66C9E07F: G***, kibuzzard-66C9E07F, B.Cu at (167.0, 138.2)
- added kibuzzard-66C9E09D: G***, kibuzzard-66C9E09D, B.Cu at (146.2, 137.6)
- added kibuzzard-66C9E0B9: G***, kibuzzard-66C9E0B9, B.Cu at (109.6, 130.8)
- added kibuzzard-66C9E0F4: G***, kibuzzard-66C9E0F4, B.Cu at (106.2, 103.0)
- added kibuzzard-66C9E100: G***, kibuzzard-66C9E100, B.Cu at (146.8, 104.2)
- moved TP601 71.4 mm to (117.8, 131.2)
- moved TP702 68.1 mm to (128.8, 129.4)
- moved TP701 65.9 mm to (128.6, 104.4)
- moved TP302 65.8 mm to (117.6, 114.8)
- moved TP303 64.5 mm to (118.8, 112.6)
- moved TP304 63.2 mm to (120.2, 114.8)
- moved TP301 62.3 mm to (121.2, 112.4)
- moved TP804 56.0 mm to (133.0, 113.8)
- moved TP803 56.0 mm to (133.0, 111.2)
- moved TP501 48.8 mm to (146.8, 106.0)
- moved TP801 45.5 mm to (143.4, 110.0)
- moved TP802 45.5 mm to (143.4, 112.6)
- moved TP401 38.3 mm to (157.8, 112.6)
- moved G*** 0.40 mm to (129.4, 137.6)
Routing:
- net +3V3: track 283.2 -> 289.7 mm
- net GND: track 0.00 -> 3.78 mm, vias 0 -> 401
- net /Control Buttons/BT_SELECT: track 3.08 -> 5.86 mm
- net /Accelerometer/ACC_SDA: track 15.5 -> 18.1 mm
- net /LEDs/LED_P3: track 38.7 -> 41.3 mm
- net /MCU/BTN_STRUM_UP: track 21.8 -> 23.9 mm
- net /LEDs/LED_P2: track 42.7 -> 44.1 mm
- net /MCU/CC1101_SCK: track 14.7 -> 16.1 mm
- net /MCU/CC1101_MISO: track 15.1 -> 16.3 mm
- net /MCU/CC1101_GDO0: track 20.2 -> 21.2 mm
- net /Accelerometer/ACC_INT1: track 30.4 -> 31.3 mm
- net /MCU/CC1101_GDO2: track 16.8 -> 17.6 mm
- net /MCU/BTN_STRUM_DOWN: track 25.3 -> 25.9 mm
- net /MCU/CC1101_~{CS}: track 20.1 -> 20.6 mm
- added copper zone on B.Cu, net GND
- added copper zone on F.Cu, net GND
Other:
- outline, holes or cut-outs redrawn
- board text added: "${TITLE} v${REVISION} ${CURRENT_DATE} ${COMPANY}"
- board text added: "X"
- board text added: "Y"
- board text added: "Z"
- board text removed: "Origina J601 Place"
- board text removed: "STRUM DOWN"
- board text removed: "STRUM UP"
- board text removed: "SWD"

Commit message: t:art: fixed noted reading, using 75hc165 for Input expander
Parts:
- removed R401, R411: 22k, Resistor_SMD:R_0603_1608Metric
- removed R402: 1k, Resistor_SMD:R_0603_1608Metric
- removed R403: 2k2, Resistor_SMD:R_0603_1608Metric
- removed R404, R405, R406: 3k3, Resistor_SMD:R_0603_1608Metric
- removed R407: 4k7, Resistor_SMD:R_0603_1608Metric
- removed R408: 5k6, Resistor_SMD:R_0603_1608Metric
- removed R409, R410: 10k, Resistor_SMD:R_0603_1608Metric
- added C402: 100n, Capacitor_SMD:C_0603_1608Metric, F.Cu at (162.8, 108.6)
- added TP402: TestPoint, TestPoint:TestPoint_Pad_D1.5mm, F.Cu at (152.8, 102.4)
- added U401: 74HC165, Package_SO:TSSOP-16_4.4x5mm_P0.65mm, F.Cu at (160.8, 126.0)
- added U402: 74HC165, Package_SO:TSSOP-16_4.4x5mm_P0.65mm, F.Cu at (160.8, 112.4)
- C401: value 1n -> 100n
- moved TP401 9.10 mm to (152.8, 105.0)
- moved C401 8.32 mm to (162.8, 122.2)
Connections:
- net /MCU/CC1101_MISO renamed /Notes/HC165_DO
- net /MCU/CC1101_SCK renamed /Notes/HC165_SCK
- C401 pad 1: /MCU/BTNS_NOTES -> +3V3
- TP401 pad 1: /MCU/BTNS_NOTES -> /Notes/HC165_LOAD
- U201 pad 2: unconnected-(U201-PC14-Pad2) -> /Notes/HC165_LOAD
- U201 pad 3: unconnected-(U201-PC15-Pad3) -> /Notes/HC165_~{CS}
- U201 pad 8: /MCU/BTNS_NOTES -> /MCU/POT_WHAM
- U201 pad 9: /MCU/POT_WHAM -> unconnected-(U201-PA2-Pad9)
Routing:
- net /Notes/HC165_~{CS}: track 0.00 -> 101.8 mm, vias 0 -> 6
- net /Notes/HC165_LOAD: track 0.00 -> 93.8 mm, vias 0 -> 5
- net /Notes/HC165_SCK: track 16.1 -> 99.8 mm, vias 2 -> 6
- net /Notes/HC165_DO: track 16.3 -> 98.4 mm, vias 0 -> 4
- net /MCU/BTNS_NOTES: track 53.3 -> 0.00 mm, vias 2 -> 0
- net +3V3: track 289.7 -> 316.0 mm, vias 11 -> 13
- net /Notes/HC165_DS: track 0.00 -> 19.3 mm
- net /Notes/BTN_YELLOW*: track 5.88 -> 22.5 mm, vias 0 -> 1
- net /Notes/BTN_RED*: track 5.87 -> 19.9 mm, vias 0 -> 1
- net /Notes/BTN_GREEN*: track 5.87 -> 17.4 mm, vias 0 -> 1
- net /Notes/BTN_ORANGE: track 5.87 -> 14.5 mm, vias 0 -> 1
- net /Notes/BTN_GREEN: track 2.68 -> 10.7 mm
- net /Notes/BTN_RED: track 5.85 -> 8.97 mm
- net /MCU/POT_WHAM: track 42.5 -> 44.1 mm
- net /Notes/BTN_YELLOW: track 5.86 -> 7.27 mm
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