File: Antares-Transmitter.kicad_pcb (KiCad board)
At the start: 2 copper layers, 94 x 60.8 mm, 99 parts, among them J1001 Debugger Pin, J1101 Conn_01x02, J401 Conn_01x11, J501 Conn_01x03, J601 Conn_01x05, J602 Conn_01x06, J901 Conn_01x05, SW701 DOWN, SW702 UP, U201 STM32G070KBTx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

Commit message: :minidisc: fixed some silkscreen, added vias and updated LCSC PNs with Basic components
Parts:
- moved TP303 0.28 mm to (118.6, 112.4)
Routing:
- net GND: track 3.78 -> 4.72 mm, vias 419 -> 443
