File: accelerometer.kicad_sch (KiCad schematic)
At the start: 9 parts, among them U801 LIS3DHTR

Commit message: :package: finished version 1.0.0, generated production files
Parts:
- gave numbers to parts that had none: 4
Changed lines of the file:
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@@
 		(on_board yes)
 		(dnp no)
-		(property "Reference" "TP?"
+		(property "Reference" "TP801"
 			(at 109.22 97.79 0)
 			(effects
@@
 			(project "Antares-Transmitter"
 				(path "/7eacce39-bbdf-4759-aeb5-d69ccfcb7b29/e5284cc2-b5aa-4898-b9b8-ce7b1c8c2af5"
-					(reference "TP?")
+					(reference "TP801")
 					(unit 1)
 				)
@@
 		(on_board yes)
 		(dnp no)
-		(property "Reference" "TP?"
+		(property "Reference" "TP802"
 			(at 115.57 97.79 0)
 			(effects
@@
 			(project "Antares-Transmitter"
 				(path "/7eacce39-bbdf-4759-aeb5-d69ccfcb7b29/e5284cc2-b5aa-4898-b9b8-ce7b1c8c2af5"
-					(reference "TP?")
+					(reference "TP802")
 					(unit 1)
 				)
@@
 		(on_board yes)
 		(dnp no)
-		(property "Reference" "TP?"
+		(property "Reference" "TP803"
 			(at 120.65 97.79 0)
 			(effects
@@
 			(project "Antares-Transmitter"
 				(path "/7eacce39-bbdf-4759-aeb5-d69ccfcb7b29/e5284cc2-b5aa-4898-b9b8-ce7b1c8c2af5"
-					(reference "TP?")
+					(reference "TP803")
 					(unit 1)
 				)
@@
 		(on_board yes)
 		(dnp no)
-		(property "Reference" "TP?"
+		(property "Reference" "TP804"
 			(at 127 97.79 0)
 			(effects
@@
 			(project "Antares-Transmitter"
 				(path "/7eacce39-bbdf-4759-aeb5-d69ccfcb7b29/e5284cc2-b5aa-4898-b9b8-ce7b1c8c2af5"
-					(reference "TP?")
-					(unit 1)
-				)
+					(reference "TP804")
+					(unit 1)
+				)

Commit message: :minidisc: fixed some silkscreen, added vias and updated LCSC PNs with Basic components
Parts:
- R801, R802: LCSC C99782 -> C23162; PN RC0603FR-074K7L -> 0603WAF4701T5E
Changed lines of the file:
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@@
 		(title "Project Antares - Transmitter Schematic")
 		(date "2024-08-23")
-		(rev "1.0.1")
+		(rev "1.0.2")
 		(company "Ourobors Embedded Development")
 		(comment 1 "Pablo Jean Rozario")
@@
 			)
 		)
-		(property "LCSC" "C99782"
+		(property "LCSC" "C23162"
 			(at 135.89 101.6 0)
 			(effects
@@
 			)
 		)
-		(property "PN" "RC0603FR-074K7L"
+		(property "PN" "0603WAF4701T5E"
 			(at 135.89 101.6 0)
 			(effects
@@
 			)
 		)
-		(property "LCSC" "C99782"
+		(property "LCSC" "C23162"
 			(at 140.97 101.6 0)
 			(effects
@@
 			)
 		)
-		(property "PN" "RC0603FR-074K7L"
+		(property "PN" "0603WAF4701T5E"
 			(at 140.97 101.6 0)
 			(effects
