File: control_buttons.kicad_sch (KiCad schematic)
At the start: 14 parts, among them J601 Conn_01x05, J602 Conn_01x06

Commit message: :package: finished version 1.0.0, generated production files
Parts:
- gave numbers to parts that had none: 1
Changed lines of the file:
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@@
 		(on_board yes)
 		(dnp no)
-		(property "Reference" "TP?"
+		(property "Reference" "TP601"
 			(at 97.79 84.3279 0)
 			(effects
@@
 			(project "Antares-Transmitter"
 				(path "/7eacce39-bbdf-4759-aeb5-d69ccfcb7b29/6f7bb571-d887-412b-afba-0267762175ed"
-					(reference "TP?")
+					(reference "TP601")
 					(unit 1)
 				)

Commit message: :minidisc: fixed some silkscreen, added vias and updated LCSC PNs with Basic components
Parts:
- C601: LCSC C100040 -> C1588; PN CC0603KRX7R9BB102 -> CL10B102KB8NNNC
- R607: LCSC C99782 -> C23162; PN RC0603FR-074K7L -> 0603WAF4701T5E
Changed lines of the file:
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@@
 		(title "Project Antares - Transmitter Schematic")
 		(date "2024-08-23")
-		(rev "1.0.1")
+		(rev "1.0.2")
 		(company "Ourobors Embedded Development")
 		(comment 1 "Pablo Jean Rozario")
@@
 			)
 		)
-		(property "LCSC" "C99782"
+		(property "LCSC" "C23162"
 			(at 113.03 135.89 0)
 			(effects
@@
 			)
 		)
-		(property "PN" "RC0603FR-074K7L"
+		(property "PN" "0603WAF4701T5E"
 			(at 113.03 135.89 0)
 			(effects
@@
 			)
 		)
-		(property "LCSC" "C100040"
+		(property "LCSC" "C1588"
 			(at 100.33 100.33 0)
 			(effects
@@
 			)
 		)
-		(property "PN" "CC0603KRX7R9BB102"
+		(property "PN" "CL10B102KB8NNNC"
 			(at 100.33 100.33 0)
 			(effects

Commit message: small fixes
Parts:
- J601: footprint Connector_JST:JST_XA_S05B-XASK-1_1x05_P2.50mm_Horizontal -> Connector_JST:JST_XH_S5B-XH-A-1_1x05_P2.50mm_Horizontal
