File: mcu.kicad_sch (KiCad schematic)
At the start: 4 parts, among them U201 STM32G070KBTx

Commit message: t:art: fixed noted reading, using 75hc165 for Input expander
Connections:
- net BTNS_NOTES is gone; now on net POT_WHAM: U201.8 (PA1)
- net POT_WHAM: no longer U201.9 (PA2)
- net BTNS_~{LD}: now reaches U201.2 (PC14)
- net BTNS_~{CS}: now reaches U201.3 (PC15)
Changed lines of the file:
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@@
 		(title "Project Antares - Transmitter Schematic")
 		(date "2024-08-23")
-		(rev "1.0.0")
+		(rev "1.0.1")
 		(company "Ourobors Embedded Development")
 		(comment 1 "Pablo Jean Rozario")
@@
 	(wire
 		(pts
-			(xy 119.38 96.52) (xy 134.62 96.52)
-		)
-		(stroke
-			(width 0)
-			(type default)
-		)
-	)
-	(wire
-		(pts
 			(xy 119.38 93.98) (xy 134.62 93.98)
 		)
@@
 	(wire
 		(pts
+			(xy 162.56 101.6) (xy 175.26 101.6)
+		)
+		(stroke
+			(width 0)
+			(type default)
+		)
+	)
+	(wire
+		(pts
 			(xy 119.38 111.76) (xy 134.62 111.76)
 		)
@@
 		(pts
 			(xy 119.38 124.46) (xy 134.62 124.46)
+		)
+		(stroke
+			(width 0)
+			(type default)
+		)
+	)
+	(wire
+		(pts
+			(xy 162.56 99.06) (xy 175.26 99.06)
 		)
 		(stroke
@@
 		)
 	)
+	(hierarchical_label "BTNS_~{CS}"
+		(shape input)
+		(at 175.26 101.6 0)
+		(fields_autoplaced yes)
+		(effects
+			(font
+				(size 1.27 1.27)
+				(color 132 0 132 1)
+			)
+			(justify left)
+		)
+	)
 	(hierarchical_label "CC1101_~{CS}"
 		(shape output)
@@
 				(size 1.27 1.27)
 				(color 204 102 0 1)
-			)
-			(justify right)
-		)
-	)
-	(hierarchical_label "POT_WHAM"
-		(shape input)
-		(at 119.38 96.52 180)
-		(fields_autoplaced yes)
-		(effects
-			(font
-				(size 1.27 1.27)
-				(color 0 0 194 1)
 			)
 			(justify right)
@@
 		)
 	)
+	(hierarchical_label "BTNS_~{LD}"
+		(shape input)
+		(at 175.26 99.06 0)
+		(fields_autoplaced yes)
+		(effects
+			(font
+				(size 1.27 1.27)
+				(color 132 0 132 1)
+			)
+			(justify left)
+		)
+	)
 	(hierarchical_label "BTN_STRUM_DOWN"
 		(shape input)
@@
 		)
 	)
+	(hierarchical_label "POT_WHAM"
+		(shape input)
+		(at 119.38 93.98 180)
+		(fields_autoplaced yes)
+		(effects
+			(font
+				(size 1.27 1.27)
+				(color 0 0 194 1)
+			)
+			(justify right)
+		)
+	)
 	(hierarchical_label "ACC_INT2"
 		(shape input)
@@
 			)
 			(justify right)
-		)
-	)
-	(hierarchical_label "BTNS_NOTES"
-		(shape input)
-		(at 119.38 93.98 180)
-		(fields_autoplaced yes)
-		(effects
-			(font
-				(size 1.27 1.27)
-				(color 132 0 132 1)
-			)
-			(justify right)

Commit message: :memo: added schematic model
Parts:
- C203: LCSC C106245 -> C1634; PN CC0603JRNPO9BN100 -> CL10C100JB8NNNC
Changed lines of the file:
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@@
 			)
 		)
-		(property "LCSC" "C106245"
+		(property "LCSC" "C1634"
 			(at 71.12 49.53 0)
 			(effects
@@
 			)
 		)
-		(property "PN" "CC0603JRNPO9BN100"
+		(property "PN" "CL10C100JB8NNNC"
 			(at 71.12 49.53 0)
 			(effects
