File: power.kicad_sch (KiCad schematic)
At the start: 3 parts, among them J1101 Conn_01x02

Commit message: small fixes
Parts:
- J1101: footprint Connector_JST:JST_XA_S02B-XASK-1_1x02_P2.50mm_Horizontal -> Connector_JST:JST_XH_S2B-XH-A-1_1x02_P2.50mm_Horizontal
Changed lines of the file:
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@@
 (kicad_sch
-	(version 20231120)
+	(version 20250114)
 	(generator "eeschema")
-	(generator_version "8.0")
+	(generator_version "9.0")
 	(paper "A4")
 	(title_block
@@
 			)
 		)
-		(property "Footprint" "Connector_JST:JST_XA_S02B-XASK-1_1x02_P2.50mm_Horizontal"
+		(property "Footprint" "Connector_JST:JST_XH_S2B-XH-A-1_1x02_P2.50mm_Horizontal"
 			(at 102.87 71.12 0)
 			(effects
