File: strum.kicad_sch (KiCad schematic)
At the start: 10 parts, among them SW701 DOWN, SW702 UP

Commit message: :package: finished version 1.0.0, generated production files
Parts:
- gave numbers to parts that had none: 2
Changed lines of the file:
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@@
 		(on_board yes)
 		(dnp no)
-		(property "Reference" "TP?"
+		(property "Reference" "TP701"
 			(at 110.49 100.8379 0)
 			(effects
@@
 			(project "Antares-Transmitter"
 				(path "/7eacce39-bbdf-4759-aeb5-d69ccfcb7b29/e897e552-39a5-4897-97b5-99c86deab657"
-					(reference "TP?")
+					(reference "TP701")
 					(unit 1)
 				)
@@
 		(on_board yes)
 		(dnp no)
-		(property "Reference" "TP?"
+		(property "Reference" "TP702"
 			(at 111.76 71.6279 0)
 			(effects
@@
 			(project "Antares-Transmitter"
 				(path "/7eacce39-bbdf-4759-aeb5-d69ccfcb7b29/e897e552-39a5-4897-97b5-99c86deab657"
-					(reference "TP?")
-					(unit 1)
-				)
+					(reference "TP702")
+					(unit 1)
+				)
